Commit message: upload my own turtlebot3
modeling finished but have to test dynamic test. There is a error about going forward
모델링 완성. 역학적 테스트 해야함. 전진 문제가 있음.

File: my_simulations/urdf/turtlebot3_my_model.urdf.xacro (robot description, xacro)
@@ -7,11 +7,11 @@
         <parent link="base_footprint"/>
         <child link="base_link" />
-        <origin xyz="0 0 0.010" rpy="0 0 0"/>
+        <origin xyz="0 0 0.060" rpy="0 0 0"/> <!-- Initial point -->
     </joint>
     <!-- Deliver robot Base -->
     <link name="base_link">
         <visual>
-            <!-- refer sdf ignore z-->
-            <origin xyz="0 0 0" rpy="0 0 0"/>
+            <!-- refer sdf (Initial point reference point)-->
+            <origin xyz="0 0 0.0" rpy="0 0 0"/>
             <geometry>
                 <box size="0.265 0.265 0.1"/>
@@ -20,13 +20,13 @@
         </visual>
         <collision>
-        <!-- refer sdf ignore z-->
-        <origin xyz="0 0 0.06" rpy="0 0 0"/>
-        <geometry>
-            <!-- refer sdf ignore z-->
-            <box size="0.265 0.265 0.1"/>
-        </geometry>
+            <!-- refer sdf(Initial point reference point) -->
+            <origin xyz="0 0 0" rpy="0 0 0"/>
+            <geometry>
+                <!-- refer sdf(Initial point reference point) -->
+                <box size="0.265 0.265 0.1"/>
+            </geometry>
         </collision>
         <inertial>
-            <origin xyz="0 0 0" rpy="0 0 0"/>
+            <origin xyz="0 0 0.0" rpy="0 0 0"/>
             <mass value="1.3729096e+00"/>
             <inertia ixx="8.7002718e-03" ixy="-4.7576583e-05" ixz="1.1160499e-04"
@@ -35,15 +35,45 @@
         </inertial>
     </link>
+    <!-- Deliver robot Caster-->
+    <!-- refer sdf (Initial point reference point)-->
+    <joint name="caster_back_joint" type="fixed">
+        <parent link="base_link"/>
+        <child link="caster_back_link"/>
+        <origin xyz="-0.11 0 -0.055" rpy="0 0 0"/>
+    </joint>
+    <link name="caster_back_link">
+        <visual>
+            <!-- refer sdf (Initial point reference point)-->
+            <origin xyz="0 0 0" rpy="0 0 0"/>
+            <geometry>
+                <sphere radius="0.005"/>
+            </geometry>
+            <material name="light_black"/>
+        </visual>
+        <collision>
+            <origin xyz="0 0 0" rpy="0 0 0"/>
+            <geometry>
+                <sphere radius="0.005"/>
+            </geometry>
+        </collision>
+        <inertial>
+            <origin xyz="0 0 0" />
+            <mass value="0.005" />
+            <inertia ixx="0.001" ixy="0.0" ixz="0.0"
+                    iyy="0.001" iyz="0.0"
+                    izz="0.001" />
+        </inertial>
+    </link>
     <!-- Deliver robot Left Wheel-->
-    <!-- refer sdf ignore z-->
+    <!-- refer sdf (Initial point reference point)-->
     <joint name="wheel_left_joint" type="continuous">
         <parent link="base_link"/>
         <child link="wheel_left_link"/>
-        <origin xyz="0.07 0.11 0.033" rpy="-1.57 0 0"/>
+        <origin xyz="0.07 0.11 -0.027" rpy="-1.57 0 0"/>
         <axis xyz="0 0 1"/>
     </joint>
     <link name="wheel_left_link">
         <visual>
-            <origin xyz="0.07 0.11 0" rpy="-1.57 0 0"/>
+            <origin xyz="0 0 0" rpy="0 0 0"/>
             <geometry>
                 <cylinder length="0.018" radius="0.033"/>
@@ -52,5 +82,5 @@
         </visual>
         <collision>
-            <origin xyz="0.07 0.11 0" rpy="0 0 0"/>
+            <origin xyz="0 0 0" rpy="0 0 0"/>
             <geometry>
                 <cylinder length="0.018" radius="0.033"/>
@@ -66,13 +96,14 @@
     </link>
     <!-- Deliver robot Right Wheel -->
+    <!-- refer sdf (Initial point reference point)-->
     <joint name="wheel_right_joint" type="continuous">
         <parent link="base_link"/>
         <child link="wheel_right_link"/>
-        <origin xyz="0.07 -0.11 0.033" rpy="-1.57 0 0"/>
+        <origin xyz="0.07 -0.11 -0.027" rpy="-1.57 0 0"/>
         <axis xyz="0 0 1"/>
     </joint>
     <link name="wheel_right_link">
         <visual>
-            <origin xyz="0.07 -0.11 0" rpy="1.57 0 0"/>
+            <origin xyz="0 0 0" rpy="0 0 0"/>
             <geometry>
                 <cylinder length="0.018" radius="0.033"/>
@@ -81,5 +112,5 @@
         </visual>
         <collision>
-            <origin xyz="0.07 -0.11 0" rpy="0 0 0"/>
+            <origin xyz="0 0 0" rpy="0 0 0"/>
             <geometry>
                 <cylinder length="0.018" radius="0.033"/>
@@ -94,37 +125,16 @@
         </inertial>
     </link>
-    <!-- Deliver robot Caster-->
-    <joint name="caster_back_joint" type="fixed">
-        <parent link="base_link"/>
-        <child link="caster_back_link"/>
-        <origin xyz="-0.11 0 0.005" rpy="-1.57 0 0"/>
-    </joint>
-    <link name="caster_back_link">
-        <collision>
-            <origin xyz="0 0.001 0" rpy="0 0 0"/>
-            <geometry>
-                <sphere radius="0.005"/>
-            </geometry>
-        </collision>
-        <inertial>
-            <origin xyz="0 0 0" />
-            <mass value="0.005" />
-            <inertia ixx="0.001" ixy="0.0" ixz="0.0"
-                    iyy="0.001" iyz="0.0"
-                    izz="0.001" />
-        </inertial>
-    </link>
     <!-- Deliver robot IMU-->
     <joint name="imu_joint" type="fixed">
         <parent link="base_link"/>
         <child link="imu_link"/>
-        <origin xyz="0.0 0 0.076" rpy="0 0 0"/>
+        <origin xyz="0.0 0 -0.048" rpy="0 0 0"/>
     </joint>
     <link name="imu_link"/>
-    <!-- Deliver robot Caster-->
+    <!-- Deliver robot scan-->
     <joint name="scan_joint" type="fixed">
         <parent link="base_link"/>
         <child link="base_scan"/>
-        <origin xyz="0 0 0.141" rpy="0 0 0"/>
+        <origin xyz="-0.012 0 0.08" rpy="0 0 0"/>
     </joint>
     <link name="base_scan">

Commit message: modeling arm(not completed)
test->have to study about arm modeling.
Do not forget to each link name and model folder name

File: my_simulations/urdf/turtlebot3_my_model.urdf.xacro (robot description, xacro)
@@ -7,5 +7,5 @@
         <parent link="base_footprint"/>
         <child link="base_link" />
-        <origin xyz="0 0 0.060" rpy="0 0 0"/> <!-- Initial point -->
+        <origin xyz="0 0 0.060" rpy="0 0 0"/> <!-- Initial point because child & parent link -->
     </joint>
     <!-- Deliver robot Base -->
@@ -29,8 +29,8 @@
         <inertial>
             <origin xyz="0 0 0.0" rpy="0 0 0"/>
-            <mass value="1.3729096e+00"/>
-            <inertia ixx="8.7002718e-03" ixy="-4.7576583e-05" ixz="1.1160499e-04"
-                    iyy="8.6195418e-03" iyz="-3.5422299e-06"
-                    izz="1.4612727e-02" />
+            <mass value="1.5"/>
+            <inertia ixx="1.0028125e-2" ixy="0" ixz="0"
+                    iyy="1.0028125e-2" iyz="0"
+                    izz="1.755625e-02" />
         </inertial>
     </link>
@@ -40,5 +40,5 @@
         <parent link="base_link"/>
         <child link="caster_back_link"/>
-        <origin xyz="-0.11 0 -0.055" rpy="0 0 0"/>
+        <origin xyz="0.11 0 -0.055" rpy="0 0 0"/>
     </joint>
     <link name="caster_back_link">
@@ -60,7 +60,7 @@
             <origin xyz="0 0 0" />
             <mass value="0.005" />
-            <inertia ixx="0.001" ixy="0.0" ixz="0.0"
-                    iyy="0.001" iyz="0.0"
-                    izz="0.001" />
+            <inertia ixx="5.0e-8" ixy="0.0" ixz="0.0"
+                    iyy="5.0e-8" iyz="0.0"
+                    izz="5.0e-8" />
         </inertial>
     </link>
@@ -70,5 +70,5 @@
         <parent link="base_link"/>
         <child link="wheel_left_link"/>
-        <origin xyz="0.07 0.11 -0.027" rpy="-1.57 0 0"/>
+        <origin xyz="-0.07 0.11 -0.027" rpy="-1.57 0 0"/>
         <axis xyz="0 0 1"/>
     </joint>
@@ -90,7 +90,7 @@
             <origin xyz="0 0 0" />
             <mass value="2.8498940e-02" />
-            <inertia ixx="1.1175580e-05" ixy="-4.2369783e-11" ixz="-5.9381719e-09"
-                    iyy="1.1192413e-05" iyz="-1.4400107e-11"
-                    izz="2.0712558e-05" />
+            <inertia ixx="1.083672194e-05" ixy="0" ixz="0"
+                    iyy="1.083672194e-05" iyz="0"
+                    izz="1.551767283e-05" />
         </inertial>
     </link>
@@ -100,5 +100,5 @@
         <parent link="base_link"/>
         <child link="wheel_right_link"/>
-        <origin xyz="0.07 -0.11 -0.027" rpy="-1.57 0 0"/>
+        <origin xyz="-0.07 -0.11 -0.027" rpy="-1.57 0 0"/>
         <axis xyz="0 0 1"/>
     </joint>
@@ -120,7 +120,7 @@
             <origin xyz="0 0 0" />
             <mass value="2.8498940e-02" />
-            <inertia ixx="1.1175580e-05" ixy="-4.2369783e-11" ixz="-5.9381719e-09"
-                    iyy="1.1192413e-05" iyz="-1.4400107e-11"
-                    izz="2.0712558e-05" />
+            <inertia ixx="1.083672194e-05" ixy="0" ixz="0"
+                    iyy="1.083672194e-05" iyz="0"
+                    izz="1.551767283e-05" />
         </inertial>
     </link>
@@ -136,5 +136,5 @@
         <parent link="base_link"/>
         <child link="base_scan"/>
-        <origin xyz="-0.012 0 0.08" rpy="0 0 0"/>
+        <origin xyz="-0.012 0 0.08" rpy="0 0 3.14"/>
     </joint>
     <link name="base_scan">
