Commit message: modeling arm completed, simulation testing
simulation testing 90% completed
robot model inertial problem have to solve

File: my_simulations/urdf/turtlebot3_my_model(backup).gazebo.xacro (robot description, xacro)
@@ -3,35 +3,4 @@
     <xacro:arg name="laser_visual"  default="false"/>
     <xacro:arg name="imu_visual"    default="false"/>
-   <!-- Init colour -->
-    <material name="black">
-        <color rgba="0.0 0.0 0.0 1.0" />
-    </material>
-    <material name="dark">
-        <color rgba="0.3 0.3 0.3 1.0" />
-    </material>
-    <material name="light_black">
-        <color rgba="0.4 0.4 0.4 1.0" />
-    </material>
-    <material name="blue">
-        <color rgba="0.0 0.0 0.8 1.0" />
-    </material>
-    <material name="green">
-        <color rgba="0.0 0.8 0.0 1.0" />
-    </material>
-    <material name="grey">
-        <color rgba="0.5 0.5 0.5 1.0" />
-    </material>
-    <material name="orange">
-        <color rgba="1.0 0.423529411765 0.0392156862745 1.0" />
-    </material>
-    <material name="brown">
-        <color rgba="0.870588235294 0.811764705882 0.764705882353 1.0" />
-    </material>
-    <material name="red">
-        <color rgba="0.8 0.0 0.0 1.0" />
-    </material>
-    <material name="white">
-        <color rgba="1.0 1.0 1.0 1.0" />
-    </material>
     <gazebo reference="base_link">
         <material>Gazebo/DarkGrey</material>
@@ -147,34 +116,34 @@
     </gazebo>
     <gazebo reference="imu_link">
-        <sensor name="imu" type="imu">
-            <always_on>true</always_on>
-            <visualize>false</visualize>
+        <sensor type="imu" name="imu">
+        <always_on>true</always_on>
+        <visualize>$(arg imu_visual)</visualize>
         </sensor>
         <material>Gazebo/FlatBlack</material>
     </gazebo>
     <gazebo>
-        <plugin filename="libgazebo_ros_diff_drive.so" name="turtlebot3_my_model_controller">
-            <commandTopic>cmd_vel</commandTopic>
-            <odometryTopic>odom</odometryTopic>
-            <odometryFrame>odom</odometryFrame>
-            <odometrySource>world</odometrySource>
-            <publishOdomTF>true</publishOdomTF>
-            <robotBaseFrame>base_footprint</robotBaseFrame>
-            <publishWheelTF>false</publishWheelTF>
-            <publishTf>true</publishTf>
-            <publishWheelJointState>true</publishWheelJointState>
-            <legacyMode>false</legacyMode>
-            <updateRate>30</updateRate>
-            <leftJoint>wheel_left_joint</leftJoint>
-            <rightJoint>wheel_right_joint</rightJoint>
-            <wheelSeparation>0.287</wheelSeparation>
-            <wheelDiameter>0.066</wheelDiameter>
-            <wheelAcceleration>1</wheelAcceleration>
-            <wheelTorque>10</wheelTorque>
-            <rosDebugLevel>na</rosDebugLevel>
+        <plugin name="turtlebot3_my_model_controller" filename="libgazebo_ros_diff_drive.so">
+        <commandTopic>cmd_vel</commandTopic>
+        <odometryTopic>odom</odometryTopic>
+        <odometryFrame>odom</odometryFrame>
+        <odometrySource>world</odometrySource>
+        <publishOdomTF>true</publishOdomTF>
+        <robotBaseFrame>base_footprint</robotBaseFrame>
+        <publishWheelTF>false</publishWheelTF>
+        <publishTf>true</publishTf>
+        <publishWheelJointState>true</publishWheelJointState>
+        <legacyMode>false</legacyMode>
+        <updateRate>30</updateRate>
+        <leftJoint>wheel_left_joint</leftJoint>
+        <rightJoint>wheel_right_joint</rightJoint>
+        <wheelSeparation>0.287</wheelSeparation>
+        <wheelDiameter>0.066</wheelDiameter>
+        <wheelAcceleration>1</wheelAcceleration>
+        <wheelTorque>10</wheelTorque>
+        <rosDebugLevel>na</rosDebugLevel>
         </plugin>
     </gazebo>
     <gazebo>
-        <plugin filename="libgazebo_ros_imu.so" name="imu_plugin">
+        <plugin name="imu_plugin" filename="libgazebo_ros_imu.so">
             <alwaysOn>true</alwaysOn>
             <bodyName>imu_link</bodyName>
@@ -205,16 +174,16 @@
     <gazebo reference="base_scan">
         <material>Gazebo/FlatBlack</material>
-        <sensor name="lds_lfcd_sensor" type="ray">
+        <sensor type="ray" name="lds_lfcd_sensor">
             <pose>0 0 0 0 0 0</pose>
-            <visualize>false</visualize>
+            <visualize>$(arg laser_visual)</visualize>
             <update_rate>5</update_rate>
             <ray>
                 <scan>
-                    <horizontal>
-                        <samples>360</samples>
-                        <resolution>1</resolution>
-                        <min_angle>0.0</min_angle>
-                        <max_angle>6.28319</max_angle>
-                    </horizontal>
+                <horizontal>
+                    <samples>360</samples>
+                    <resolution>1</resolution>
+                    <min_angle>0.0</min_angle>
+                    <max_angle>6.28319</max_angle>
+                </horizontal>
                 </scan>
                 <range>
@@ -229,5 +198,5 @@
                 </noise>
             </ray>
-            <plugin filename="libgazebo_ros_laser.so" name="gazebo_ros_lds_lfcd_controller">
+            <plugin name="gazebo_ros_lds_lfcd_controller" filename="libgazebo_ros_laser.so">
                 <topicName>scan</topicName>
                 <frameName>base_scan</frameName>
@@ -235,9 +204,3 @@
         </sensor>
     </gazebo>
-    <gazebo>
-        <plugin name="gazebo_ros_control" filename="libgazebo_ros_control.so">
-            <robotNamespace>/</robotNamespace>
-            <legacyModeNS>true</legacyModeNS>
-        </plugin>
-    </gazebo>
 </robot>

File: my_simulations/urdf/turtlebot3_my_model.urdf.xacro (robot description, xacro)
@@ -1,11 +1,15 @@
-<?xml version="1.0"?>
+<?xml version="1.0" ?>
+<!-- =================================================================================== -->
+<!-- |    This document was autogenerated by xacro from /home/duckbe/catkin_ws/src/my_simulations/urdf/turtlebot3_my_model.urdf.xacro | -->
+<!-- |    EDITING THIS FILE BY HAND IS NOT RECOMMENDED                                 | -->
+<!-- =================================================================================== -->
 <robot name="turtlebot3_my_model" xmlns:xacro="http://ros.org/wiki/xacro">
-    <xacro:include filename="$(find my_simulations)/urdf/common_properties.xacro"/>
     <xacro:include filename="$(find my_simulations)/urdf/turtlebot3_my_model.gazebo.xacro"/>
-    <link name="base_footprint"/>
+    <link name="base_footprint" />
     <joint name="base_joint" type="fixed">
-        <parent link="base_footprint"/>
+        <parent link="base_footprint" />
         <child link="base_link" />
-        <origin xyz="0 0 0.060" rpy="0 0 0"/> <!-- Initial point because child & parent link -->
+        <origin rpy="0 0 0" xyz="0 0 0.06" />
+        <!-- Initial point because child & parent link -->
     </joint>
     <!-- Deliver robot Base -->
@@ -13,24 +17,22 @@
         <visual>
             <!-- refer sdf (Initial point reference point)-->
-            <origin xyz="0 0 0.0" rpy="0 0 0"/>
-            <geometry>
-                <box size="0.265 0.265 0.1"/>
-            </geometry>
-            <material name="light_black"/>
+            <origin rpy="0 0 0" xyz="0 0 0.0" />
+            <geometry>
+                <box size="0.265 0.265 0.1" />
+            </geometry>
+            <material name="light_black" />
         </visual>
         <collision>
             <!-- refer sdf(Initial point reference point) -->
-            <origin xyz="0 0 0" rpy="0 0 0"/>
+            <origin rpy="0 0 0" xyz="0 0 0" />
             <geometry>
                 <!-- refer sdf(Initial point reference point) -->
-                <box size="0.265 0.265 0.1"/>
-            </geometry>
-        </collision>
-        <inertial>
-            <origin xyz="0 0 0.0" rpy="0 0 0"/>
-            <mass value="1.5"/>
-            <inertia ixx="1.0028125e-2" ixy="0" ixz="0"
-                    iyy="1.0028125e-2" iyz="0"
-                    izz="1.755625e-02" />
+                <box size="0.265 0.265 0.1" />
+            </geometry>
+        </collision>
+        <inertial>
+            <origin rpy="0 0 0" xyz="0 0 0.0" />
+            <mass value="1.5" />
+            <inertia ixx="1.0028125e-2" ixy="0" ixz="0" iyy="1.0028125e-2" iyz="0" izz="1.755625e-02" />
         </inertial>
     </link>
@@ -38,21 +40,21 @@
     <!-- refer sdf (Initial point reference point)-->
     <joint name="caster_back_joint" type="fixed">
-        <parent link="base_link"/>
-        <child link="caster_back_link"/>
-        <origin xyz="0.11 0 -0.055" rpy="0 0 0"/>
+        <parent link="base_link" />
+        <child link="caster_back_link" />
+        <origin rpy="0 0 0" xyz="0.11 0 -0.055" />
     </joint>
     <link name="caster_back_link">
         <visual>
             <!-- refer sdf (Initial point reference point)-->
-            <origin xyz="0 0 0" rpy="0 0 0"/>
-            <geometry>
-                <sphere radius="0.005"/>
-            </geometry>
-            <material name="light_black"/>
-        </visual>
-        <collision>
-            <origin xyz="0 0 0" rpy="0 0 0"/>
-            <geometry>
-                <sphere radius="0.005"/>
+            <origin rpy="0 0 0" xyz="0 0 0" />
+            <geometry>
+                <sphere radius="0.005" />
+            </geometry>
+            <material name="light_black" />
+        </visual>
+        <collision>
+            <origin rpy="0 0 0" xyz="0 0 0" />
+            <geometry>
+                <sphere radius="0.005" />
             </geometry>
         </collision>
@@ -60,7 +62,5 @@
             <origin xyz="0 0 0" />
             <mass value="0.005" />
-            <inertia ixx="5.0e-8" ixy="0.0" ixz="0.0"
-                    iyy="5.0e-8" iyz="0.0"
-                    izz="5.0e-8" />
+            <inertia ixx="5.0e-8" ixy="0.0" ixz="0.0" iyy="5.0e-8" iyz="0.0" izz="5.0e-8" />
         </inertial>
     </link>
@@ -68,21 +68,21 @@
     <!-- refer sdf (Initial point reference point)-->
     <joint name="wheel_left_joint" type="continuous">
-        <parent link="base_link"/>
-        <child link="wheel_left_link"/>
-        <origin xyz="-0.07 0.11 -0.027" rpy="-1.57 0 0"/>
-        <axis xyz="0 0 1"/>
+        <parent link="base_link" />
+        <child link="wheel_left_link" />
+        <origin rpy="-1.57 0 0" xyz="-0.07 0.11 -0.027" />
+        <axis xyz="0 0 1" />
     </joint>
     <link name="wheel_left_link">
         <visual>
-            <origin xyz="0 0 0" rpy="0 0 0"/>
-            <geometry>
-                <cylinder length="0.018" radius="0.033"/>
-            </geometry>
-            <material name="dark"/>
-        </visual>
-        <collision>
-            <origin xyz="0 0 0" rpy="0 0 0"/>
-            <geometry>
-                <cylinder length="0.018" radius="0.033"/>
+            <origin rpy="0 0 0" xyz="0 0 0" />
+            <geometry>
+                <cylinder length="0.018" radius="0.033" />
+            </geometry>
+            <material name="dark" />
+        </visual>
+        <collision>
+            <origin rpy="0 0 0" xyz="0 0 0" />
+            <geometry>
+                <cylinder length="0.018" radius="0.033" />
             </geometry>
         </collision>
@@ -90,7 +90,5 @@
             <origin xyz="0 0 0" />
             <mass value="2.8498940e-02" />
-            <inertia ixx="1.083672194e-05" ixy="0" ixz="0"
-                    iyy="1.083672194e-05" iyz="0"
-                    izz="1.551767283e-05" />
+            <inertia ixx="1.083672194e-05" ixy="0" ixz="0" iyy="1.083672194e-05" iyz="0" izz="1.551767283e-05" />
         </inertial>
     </link>
@@ -98,21 +96,21 @@
     <!-- refer sdf (Initial point reference point)-->
     <joint name="wheel_right_joint" type="continuous">
-        <parent link="base_link"/>
-        <child link="wheel_right_link"/>
-        <origin xyz="-0.07 -0.11 -0.027" rpy="-1.57 0 0"/>
-        <axis xyz="0 0 1"/>
+        <parent link="base_link" />
+        <child link="wheel_right_link" />
+        <origin rpy="-1.57 0 0" xyz="-0.07 -0.11 -0.027" />
+        <axis xyz="0 0 1" />
     </joint>
     <link name="wheel_right_link">
         <visual>
-            <origin xyz="0 0 0" rpy="0 0 0"/>
-            <geometry>
-                <cylinder length="0.018" radius="0.033"/>
-            </geometry>
-            <material name="dark"/>
-        </visual>
-        <collision>
-            <origin xyz="0 0 0" rpy="0 0 0"/>
-            <geometry>
-                <cylinder length="0.018" radius="0.033"/>
+            <origin rpy="0 0 0" xyz="0 0 0" />
+            <geometry>
+                <cylinder length="0.018" radius="0.033" />
+            </geometry>
+            <material name="dark" />
+        </visual>
+        <collision>
+            <origin rpy="0 0 0" xyz="0 0 0" />
+            <geometry>
+                <cylinder length="0.018" radius="0.033" />
             </geometry>
         </collision>
@@ -120,262 +118,196 @@
             <origin xyz="0 0 0" />
             <mass value="2.8498940e-02" />
-            <inertia ixx="1.083672194e-05" ixy="0" ixz="0"
-                    iyy="1.083672194e-05" iyz="0"
-                    izz="1.551767283e-05" />
+            <inertia ixx="1.083672194e-05" ixy="0" ixz="0" iyy="1.083672194e-05" iyz="0" izz="1.551767283e-05" />
         </inertial>
     </link>
     <!-- Deliver robot joint1-->
-    <joint name="joint1_left_joint" type="continuous">
-        <parent link="base_link"/>
-        <child link = "joint1_left_link"/>
-        <origin xyz="0.11 -0.135 0.04" rpy="-1.57 0 0"/>
-        <axis xyz= "0 0 1"/>
-    </joint>
-    <link name = "joint1_left_link">
-        <visual>
-            <origin xyz="0 0 0" rpy="0 0 0"/>
-            <geometry>
-                <cylinder length="0.018" radius="0.015"/>
-            </geometry>
-            <material name="dark"/>
-        </visual>
-        <collision>
-            <origin xyz="0 0 0" rpy="0 0 0"/>
-            <geometry>
-                <cylinder length="0.018" radius="0.015"/>
-            </geometry>
-        </collision>
-        <inertial>
-            <origin xyz="0 0 0"/>
-            <mass value = "0.1"/>
-            <inertia ixx="1.6425e-5" ixy="0" ixz="0"
-                    iyy="1.6425e-5" iyz="0"
-                    izz="1.125e-5"/>
-        </inertial>
-    </link>
-    <joint name="joint1_right_joint" type="continuous">
-        <parent link="base_link"/>
-        <child link = "joint1_right_link"/>
-        <origin xyz="0.11 0.135 0.04" rpy="-1.57 0 0"/>
-        <axis xyz= "0 0 1"/>
-    </joint>
-    <link name = "joint1_right_link">
-        <visual>
-            <origin xyz="0 0 0" rpy="0 0 0"/>
-            <geometry>
-                <cylinder length="0.018" radius="0.015"/>
-            </geometry>
-            <material name="dark"/>
-        </visual>
-        <collision>
-            <origin xyz="0 0 0" rpy="0 0 0"/>
-            <geometry>
-                <cylinder length="0.018" radius="0.015"/>
-            </geometry>
-        </collision>
-        <inertial>
-            <origin xyz="0 0 0"/>
-            <mass value = "0.1"/>
-            <inertia ixx="1.6425e-5" ixy="0" ixz="0"
-                    iyy="1.6425e-5" iyz="0"
-                    izz="1.125e-5"/>
-        </inertial>
-    </link>
-    <!-- Deliver robot link1-->
-    <joint name="link1_left_joint" type="continuous">
-        <parent link="joint1_left_link"/>
-        <child link = "link1_left_link"/>
-        <origin xyz="0 0 0" rpy="0 0 0"/>
-        <axis xyz= "0 0 1"/>
-    </joint>
-    <link name = "link1_left_link">
-        <visual>
-            <origin xyz="0.05 0 0" rpy="0 0 0"/>
-            <geometry>
-                <box size="0.1 0.03 0.03"/>
-            </geometry>
-            <material name="dark"/>
-        </visual>
-        <collision>
-            <origin xyz="0.05 0 0" rpy="0 0 0"/>
-            <geometry>
-                <box size="0.1 0.03 0.03"/>
-            </geometry>
-        </collision>
-        <inertial>
-            <origin xyz="0.05 0 0"/>
-            <mass value = "0.1"/>
-            <inertia ixx="1.6425e-5" ixy="0" ixz="0"
-                    iyy="1.6425e-5" iyz="0"
-                    izz="1.125e-5"/>
-        </inertial>
-    </link>
-    <joint name="link1_right_joint" type="continuous">
-        <parent link="joint1_right_link"/>
-        <child link = "link1_right_link"/>
-        <origin xyz="0 0 0" rpy="0 0 0"/>
-        <axis xyz= "0 0 1"/>
-    </joint>
-    <link name = "link1_right_link">
-        <visual>
-            <origin xyz="0.05 0 0" rpy="0 0 0"/>
-            <geometry>
-                <box size="0.1 0.03 0.03"/>
-            </geometry>
-            <material name="dark"/>
-        </visual>
-        <collision>
-            <origin xyz="0.05 0 0" rpy="0 0 0"/>
-            <geometry>
-                <box size="0.1 0.03 0.03"/>
-            </geometry>
-        </collision>
-        <inertial>
-            <origin xyz="0.05 0 0"/>
-            <mass value = "0.1"/>
-            <inertia ixx="1.6425e-5" ixy="0" ixz="0"
-                    iyy="1.6425e-5" iyz="0"
-                    izz="1.125e-5"/>
+    <joint name="joint1_left_joint" type="revolute">
+        <!--revolute have to limit-->
+        <parent link="base_link" />
+        <child link="joint1_left_link" />
+        <origin rpy="-1.57 0 0" xyz="0.11 -0.135 0.04" />
+        <axis xyz="0 0 1" />
+        <!--Force, degree max min, velocity-->
+        <limit effort="3" lower="-2.617" upper="2.617" velocity="0.05" />
+    </joint>
+    <link name="joint1_left_link">
+        <visual>
+            <origin rpy="0 0 0" xyz="0 0 0" />
+            <geometry>
+                <cylinder length="0.018" radius="0.015" />
+            </geometry>
+            <material name="dark" />
+        </visual>
+        <collision>
+            <origin rpy="0 0 0" xyz="0 0 0" />
+            <geometry>
+                <cylinder length="0.018" radius="0.015" />
+            </geometry>
+        </collision>
+        <visual>
+            <origin rpy="0 0 0" xyz="0.05 0 0" />
+            <geometry>
+                <box size="0.1 0.03 0.03" />
+            </geometry>
+            <material name="dark" />
+        </visual>
+        <collision>
+            <origin rpy="0 0 0" xyz="0.05 0 0" />
+            <geometry>
+                <box size="0.1 0.03 0.03" />
+            </geometry>
+        </collision>
+        <inertial>
+            <origin xyz="0.05 0 0" />
+            <mass value="0.01" />
+            <inertia ixx="1.6425e-6" ixy="0" ixz="0" iyy="1.6425e-6" iyz="0" izz="1.125e-6" />
+        </inertial>
+    </link>
+    <joint name="joint1_right_joint" type="revolute">
+        <parent link="base_link" />
+        <child link="joint1_right_link" />
+        <origin rpy="-1.57 0 0" xyz="0.11 0.135 0.04" />
+        <axis xyz="0 0 1" />
+        <limit effort="3" lower="-2.617" upper="2.617" velocity="0.05" />
+    </joint>
+    <link name="joint1_right_link">
+        <visual>
+            <origin rpy="0 0 0" xyz="0 0 0" />
+            <geometry>
+                <cylinder length="0.018" radius="0.015" />
+            </geometry>
+            <material name="dark" />
+        </visual>
+        <collision>
+            <origin rpy="0 0 0" xyz="0 0 0" />
+            <geometry>
+                <cylinder length="0.018" radius="0.015" />
+            </geometry>
+        </collision>
+        <visual>
+            <origin rpy="0 0 0" xyz="0.05 0 0" />
+            <geometry>
+                <box size="0.1 0.03 0.03" />
+            </geometry>
+            <material name="dark" />
+        </visual>
+        <collision>
+            <origin rpy="0 0 0" xyz="0.05 0 0" />
+            <geometry>
+                <box size="0.1 0.03 0.03" />
+            </geometry>
+        </collision>
+        <inertial>
+            <origin xyz="0.05 0 0" />
+            <mass value="0.01" />
+            <inertia ixx="1.6425e-6" ixy="0" ixz="0" iyy="1.6425e-6" iyz="0" izz="1.125e-6" />
         </inertial>
     </link>
     <!-- Deliver robot joint2-->
-    <joint name="joint2_left_joint" type="continuous">
-        <parent link="link1_left_link"/>
-        <child link = "joint2_left_link"/>
-        <origin xyz="0.1 0 0" rpy="0 0 0"/>
-        <axis xyz= "0 0 1"/>
-    </joint>
-    <link name = "joint2_left_link">
-        <visual>
-            <origin xyz="0 0 0" rpy="0 0 0"/>
-            <geometry>
-                <cylinder length="0.018" radius="0.015"/>
-            </geometry>
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