Commit message: urdf modeling completed
urdf robot arm modeling completed

File: my_simulations/urdf/turtlebot3_my_model.gazebo.xacro (robot description, xacro)
@@ -33,4 +33,84 @@
         <minDepth>0.001</minDepth>
         <maxVel>1.0</maxVel>
+        <material>Gazebo/FlatBlack</material>
+    </gazebo>
+    <gazebo reference="joint1_left_link">
+        <mu1>0.1</mu1>
+        <mu2>0.1</mu2>
+        <kp>500000.0</kp>
+        <kd>10.0</kd>
+        <minDepth>0.001</minDepth>
+        <maxVel>0.1</maxVel>
+        <fdir1>1 0 0</fdir1>
+        <material>Gazebo/FlatBlack</material>
+    </gazebo>
+    <gazebo reference="joint1_right_link">
+        <mu1>0.1</mu1>
+        <mu2>0.1</mu2>
+        <kp>500000.0</kp>
+        <kd>10.0</kd>
+        <minDepth>0.001</minDepth>
+        <maxVel>0.1</maxVel>
+        <fdir1>1 0 0</fdir1>
+        <material>Gazebo/FlatBlack</material>
+    </gazebo>
+    <gazebo reference="link1_left_link">
+        <mu1>0.1</mu1>
+        <mu2>0.1</mu2>
+        <kp>500000.0</kp>
+        <kd>10.0</kd>
+        <minDepth>0.001</minDepth>
+        <maxVel>0.1</maxVel>
+        <fdir1>1 0 0</fdir1>
+        <material>Gazebo/FlatBlack</material>
+    </gazebo>
+    <gazebo reference="link1_right_link">
+        <mu1>0.1</mu1>
+        <mu2>0.1</mu2>
+        <kp>500000.0</kp>
+        <kd>10.0</kd>
+        <minDepth>0.001</minDepth>
+        <maxVel>0.1</maxVel>
+        <fdir1>1 0 0</fdir1>
+        <material>Gazebo/FlatBlack</material>
+    </gazebo>
+    <gazebo reference="joint2_left_link">
+        <mu1>0.1</mu1>
+        <mu2>0.1</mu2>
+        <kp>500000.0</kp>
+        <kd>10.0</kd>
+        <minDepth>0.001</minDepth>
+        <maxVel>0.1</maxVel>
+        <fdir1>1 0 0</fdir1>
+        <material>Gazebo/FlatBlack</material>
+    </gazebo>
+    <gazebo reference="joint2_right_link">
+        <mu1>0.1</mu1>
+        <mu2>0.1</mu2>
+        <kp>500000.0</kp>
+        <kd>10.0</kd>
+        <minDepth>0.001</minDepth>
+        <maxVel>0.1</maxVel>
+        <fdir1>1 0 0</fdir1>
+        <material>Gazebo/FlatBlack</material>
+    </gazebo>
+    <gazebo reference="link2_left_link">
+        <mu1>0.1</mu1>
+        <mu2>0.1</mu2>
+        <kp>500000.0</kp>
+        <kd>10.0</kd>
+        <minDepth>0.001</minDepth>
+        <maxVel>0.1</maxVel>
+        <fdir1>1 0 0</fdir1>
+        <material>Gazebo/FlatBlack</material>
+    </gazebo>
+    <gazebo reference="link2_right_link">
+        <mu1>0.1</mu1>
+        <mu2>0.1</mu2>
+        <kp>500000.0</kp>
+        <kd>10.0</kd>
+        <minDepth>0.001</minDepth>
+        <maxVel>0.1</maxVel>
+        <fdir1>1 0 0</fdir1>
         <material>Gazebo/FlatBlack</material>
     </gazebo>

File: my_simulations/urdf/turtlebot3_my_model.urdf.xacro (robot description, xacro)
@@ -125,4 +125,232 @@
         </inertial>
     </link>
+    <!-- Deliver robot joint1-->
+    <joint name="joint1_left_joint" type="continuous">
+        <parent link="base_link"/>
+        <child link = "joint1_left_link"/>
+        <origin xyz="0.11 -0.135 0.04" rpy="-1.57 0 0"/>
+        <axis xyz= "0 0 1"/>
+    </joint>
+    <link name = "joint1_left_link">
+        <visual>
+            <origin xyz="0 0 0" rpy="0 0 0"/>
+            <geometry>
+                <cylinder length="0.018" radius="0.015"/>
+            </geometry>
+            <material name="dark"/>
+        </visual>
+        <collision>
+            <origin xyz="0 0 0" rpy="0 0 0"/>
+            <geometry>
+                <cylinder length="0.018" radius="0.015"/>
+            </geometry>
+        </collision>
+        <inertial>
+            <origin xyz="0 0 0"/>
+            <mass value = "0.1"/>
+            <inertia ixx="1.6425e-5" ixy="0" ixz="0"
+                    iyy="1.6425e-5" iyz="0"
+                    izz="1.125e-5"/>
+        </inertial>
+    </link>
+    <joint name="joint1_right_joint" type="continuous">
+        <parent link="base_link"/>
+        <child link = "joint1_right_link"/>
+        <origin xyz="0.11 0.135 0.04" rpy="-1.57 0 0"/>
+        <axis xyz= "0 0 1"/>
+    </joint>
+    <link name = "joint1_right_link">
+        <visual>
+            <origin xyz="0 0 0" rpy="0 0 0"/>
+            <geometry>
+                <cylinder length="0.018" radius="0.015"/>
+            </geometry>
+            <material name="dark"/>
+        </visual>
+        <collision>
+            <origin xyz="0 0 0" rpy="0 0 0"/>
+            <geometry>
+                <cylinder length="0.018" radius="0.015"/>
+            </geometry>
+        </collision>
+        <inertial>
+            <origin xyz="0 0 0"/>
+            <mass value = "0.1"/>
+            <inertia ixx="1.6425e-5" ixy="0" ixz="0"
+                    iyy="1.6425e-5" iyz="0"
+                    izz="1.125e-5"/>
+        </inertial>
+    </link>
+    <!-- Deliver robot link1-->
+    <joint name="link1_left_joint" type="continuous">
+        <parent link="joint1_left_link"/>
+        <child link = "link1_left_link"/>
+        <origin xyz="0 0 0" rpy="0 0 0"/>
+        <axis xyz= "0 0 1"/>
+    </joint>
+    <link name = "link1_left_link">
+        <visual>
+            <origin xyz="0.05 0 0" rpy="0 0 0"/>
+            <geometry>
+                <box size="0.1 0.03 0.03"/>
+            </geometry>
+            <material name="dark"/>
+        </visual>
+        <collision>
+            <origin xyz="0.05 0 0" rpy="0 0 0"/>
+            <geometry>
+                <box size="0.1 0.03 0.03"/>
+            </geometry>
+        </collision>
+        <inertial>
+            <origin xyz="0.05 0 0"/>
+            <mass value = "0.1"/>
+            <inertia ixx="1.6425e-5" ixy="0" ixz="0"
+                    iyy="1.6425e-5" iyz="0"
+                    izz="1.125e-5"/>
+        </inertial>
+    </link>
+    <joint name="link1_right_joint" type="continuous">
+        <parent link="joint1_right_link"/>
+        <child link = "link1_right_link"/>
+        <origin xyz="0 0 0" rpy="0 0 0"/>
+        <axis xyz= "0 0 1"/>
+    </joint>
+    <link name = "link1_right_link">
+        <visual>
+            <origin xyz="0.05 0 0" rpy="0 0 0"/>
+            <geometry>
+                <box size="0.1 0.03 0.03"/>
+            </geometry>
+            <material name="dark"/>
+        </visual>
+        <collision>
+            <origin xyz="0.05 0 0" rpy="0 0 0"/>
+            <geometry>
+                <box size="0.1 0.03 0.03"/>
+            </geometry>
+        </collision>
+        <inertial>
+            <origin xyz="0.05 0 0"/>
+            <mass value = "0.1"/>
+            <inertia ixx="1.6425e-5" ixy="0" ixz="0"
+                    iyy="1.6425e-5" iyz="0"
+                    izz="1.125e-5"/>
+        </inertial>
+    </link>
+    <!-- Deliver robot joint2-->
+    <joint name="joint2_left_joint" type="continuous">
+        <parent link="link1_left_link"/>
+        <child link = "joint2_left_link"/>
+        <origin xyz="0.1 0 0" rpy="0 0 0"/>
+        <axis xyz= "0 0 1"/>
+    </joint>
+    <link name = "joint2_left_link">
+        <visual>
+            <origin xyz="0 0 0" rpy="0 0 0"/>
+            <geometry>
+                <cylinder length="0.018" radius="0.015"/>
+            </geometry>
+            <material name="dark"/>
+        </visual>
+        <collision>
+            <origin xyz="0 0 0" rpy="0 0 0"/>
+            <geometry>
+                <cylinder length="0.018" radius="0.015"/>
+            </geometry>
+        </collision>
+        <inertial>
+            <origin xyz="0 0 0"/>
+            <mass value = "0.1"/>
+            <inertia ixx="1.6425e-5" ixy="0" ixz="0"
+                    iyy="1.6425e-5" iyz="0"
+                    izz="1.125e-5"/>
+        </inertial>
+    </link>
+    <joint name="joint2_right_joint" type="continuous">
+        <parent link="link1_right_link"/>
+        <child link = "joint2_right_link"/>
+        <origin xyz="0.1 0 0" rpy="0 0 0"/>
+        <axis xyz="0 0 1"/>
+    </joint>
+    <link name = "joint2_right_link">
+        <visual>
+            <origin xyz="0 0 0" rpy="0 0 0"/>
+            <geometry>
+                <cylinder length="0.018" radius="0.015"/>
+            </geometry>
+            <material name="dark"/>
+        </visual>
+        <collision>
+            <origin xyz="0 0 0" rpy="0 0 0"/>
+            <geometry>
+                <cylinder length="0.018" radius="0.015"/>
+            </geometry>
+        </collision>
+        <inertial>
+            <origin xyz="0 0 0"/>
+            <mass value = "0.1"/>
+            <inertia ixx="1.6425e-5" ixy="0" ixz="0"
+                    iyy="1.6425e-5" iyz="0"
+                    izz="1.125e-5"/>
+        </inertial>
+    </link>
+    <!-- Deliver robot link2-->
+    <joint name="link2_left_joint" type="continuous">
+        <parent link="joint2_left_link"/>
+        <child link = "link2_left_link"/>
+        <origin xyz="0 0 0" rpy="0 0 0"/>
+        <axis xyz= "0 0 1"/>
+    </joint>
+    <link name = "link2_left_link">
+        <visual>
+            <origin xyz="0.05 0 0" rpy="0 0 0"/>
+            <geometry>
+                <box size="0.1 0.03 0.03"/>
+            </geometry>
+            <material name="dark"/>
+        </visual>
+        <collision>
+            <origin xyz="0.05 0 0" rpy="0 0 0"/>
+            <geometry>
+                <box size="0.1 0.03 0.03"/>
+            </geometry>
+        </collision>
+        <inertial>
+            <origin xyz="0.05 0 0"/>
+            <mass value = "0.1"/>
+            <inertia ixx="1.6425e-5" ixy="0" ixz="0"
+                    iyy="1.6425e-5" iyz="0"
+                    izz="1.125e-5"/>
+        </inertial>
+    </link>
+    <joint name="link2_right_joint" type="continuous">
+        <parent link="joint2_right_link"/>
+        <child link = "link2_right_link"/>
+        <origin xyz="0 0 0" rpy="0 0 0"/>
+        <axis xyz= "0 0 1"/>
+    </joint>
+    <link name = "link2_right_link">
+        <visual>
+            <origin xyz="0.05 0 0" rpy="0 0 0"/>
+            <geometry>
+                <box size="0.1 0.03 0.03"/>
+            </geometry>
+            <material name="dark"/>
+        </visual>
+        <collision>
+            <origin xyz="0.05 0 0" rpy="0 0 0"/>
+            <geometry>
+                <box size="0.1 0.03 0.03"/>
+            </geometry>
+        </collision>
+        <inertial>
+            <origin xyz="0.05 0 0"/>
+            <mass value = "0.1"/>
+            <inertia ixx="1.6425e-5" ixy="0" ixz="0"
+                    iyy="1.6425e-5" iyz="0"
+                    izz="1.125e-5"/>
+        </inertial>
+    </link>
     <!-- Deliver robot IMU-->
     <joint name="imu_joint" type="fixed">

Commit message: solving dynamic problem but not completed

File: my_simulations/urdf/turtlebot3_my_model.gazebo.xacro (robot description, xacro)
@@ -72,5 +72,5 @@
         <kd>10.0</kd>
         <minDepth>0.001</minDepth>
-        <maxVel>0.1</maxVel>
+        <maxVel>0.05</maxVel>
         <fdir1>1 0 0</fdir1>
         <material>Gazebo/FlatBlack</material>
@@ -82,5 +82,5 @@
         <kd>10.0</kd>
         <minDepth>0.001</minDepth>
-        <maxVel>0.1</maxVel>
+        <maxVel>0.05</maxVel>
         <fdir1>1 0 0</fdir1>
         <material>Gazebo/FlatBlack</material>
@@ -92,5 +92,5 @@
         <kd>10.0</kd>
         <minDepth>0.001</minDepth>
-        <maxVel>0.1</maxVel>
+        <maxVel>0.05</maxVel>
         <fdir1>1 0 0</fdir1>
         <material>Gazebo/FlatBlack</material>
@@ -102,5 +102,5 @@
         <kd>10.0</kd>
         <minDepth>0.001</minDepth>
-        <maxVel>0.1</maxVel>
+        <maxVel>0.05</maxVel>
         <fdir1>1 0 0</fdir1>
         <material>Gazebo/FlatBlack</material>
@@ -112,5 +112,5 @@
         <kd>10.0</kd>
         <minDepth>0.001</minDepth>
-        <maxVel>0.1</maxVel>
+        <maxVel>0.05</maxVel>
         <fdir1>1 0 0</fdir1>
         <material>Gazebo/FlatBlack</material>
@@ -122,5 +122,5 @@
         <kd>10.0</kd>
         <minDepth>0.001</minDepth>
-        <maxVel>0.1</maxVel>
+        <maxVel>0.05</maxVel>
         <fdir1>1 0 0</fdir1>
         <material>Gazebo/FlatBlack</material>
@@ -132,5 +132,5 @@
         <kd>10.0</kd>
         <minDepth>0.001</minDepth>
-        <maxVel>0.1</maxVel>
+        <maxVel>0.05</maxVel>
         <fdir1>1 0 0</fdir1>
         <material>Gazebo/FlatBlack</material>
@@ -142,5 +142,5 @@
         <kd>10.0</kd>
         <minDepth>0.001</minDepth>
-        <maxVel>0.1</maxVel>
+        <maxVel>0.05</maxVel>
         <fdir1>1 0 0</fdir1>
         <material>Gazebo/FlatBlack</material>

File: my_simulations/urdf/turtlebot3_my_model.urdf.xacro (robot description, xacro)
@@ -34,5 +34,7 @@
             <origin rpy="0 0 0" xyz="0 0 0.0" />
             <mass value="1.5" />
-            <inertia ixx="1.0028125e-2" ixy="0" ixz="0" iyy="1.0028125e-2" iyz="0" izz="1.755625e-02" />
+            <inertia ixx="8.7002718e-03" ixy="-4.7576583e-05" ixz="1.1160499e-04"
+                    iyy="8.6195418e-03" iyz="-3.5422299e-06"
+                    izz="1.4612727e-02" />
         </inertial>
     </link>
@@ -62,5 +64,7 @@
             <origin xyz="0 0 0" />
             <mass value="0.005" />
-            <inertia ixx="5.0e-8" ixy="0.0" ixz="0.0" iyy="5.0e-8" iyz="0.0" izz="5.0e-8" />
+            <inertia ixx="0.001" ixy="0.0" ixz="0.0"
+                    iyy="0.001" iyz="0.0"
+                    izz="0.001" />
         </inertial>
     </link>
@@ -90,5 +94,7 @@
             <origin xyz="0 0 0" />
             <mass value="2.8498940e-02" />
-            <inertia ixx="1.083672194e-05" ixy="0" ixz="0" iyy="1.083672194e-05" iyz="0" izz="1.551767283e-05" />
+            <inertia ixx="1.1175580e-05" ixy="-4.2369783e-11" ixz="-5.9381719e-09"
+                    iyy="1.1192413e-05" iyz="-1.4400107e-11"
+                    izz="2.0712558e-05" />
         </inertial>
     </link>
@@ -118,5 +124,7 @@
             <origin xyz="0 0 0" />
             <mass value="2.8498940e-02" />
-            <inertia ixx="1.083672194e-05" ixy="0" ixz="0" iyy="1.083672194e-05" iyz="0" izz="1.551767283e-05" />
+            <inertia ixx="1.1175580e-05" ixy="-4.2369783e-11" ixz="-5.9381719e-09"
+                    iyy="1.1192413e-05" iyz="-1.4400107e-11"
+                    izz="2.0712558e-05" />
         </inertial>
     </link>
